File: cad/led_bage.kicad_pcb (KiCad board)
At the start: 4 copper layers, 72.6 x 123.7 mm, 3254 parts, among them J1 Conn_01x08_Socket, J2 Conn_01x08_Socket, Q2 AO4407A, Q3 AO4407A, Q4 AO4407A, Q5 AO4407A, Q6 AO4407A, Q7 AO4407A, Q8 AO4407A, Q9 AO4407A, U2 74AHCT1G125, U3 74AHCT1G125, U4 74AHCT1G125, U5 74AHCT1G125, U6 74AHCT1G125, U7 74AHCT1G125, U8 74AHCT1G125, U9 74AHCT1G125

Commit message: feat: scale protection circuit toward 2500-LED main board
Add Si7145DP P-FET (U1) and SnapEDA-imported library table (fp-lib-table)
to the main board. WIP: U1 pin-to-net mapping is incorrect — drain pads
currently land on VDD instead of VDD_S, so the FET is shorted across
itself and not actually protecting anything yet.

Add three pcbnew automation scripts to support the build:
- stitch_power_planes.py: checkerboard via stitching across In1.Cu/In2.Cu
- add_thermal_vias.py: drops thermal via grid under exposed pads
- place_bulk_caps.py: clones a template cap across the LED bbox

Sample board updated alongside the main board for prototyping continuity.
Parts:
- removed J2: Conn_01x08_Socket, Connector_Molex:Molex_CLIK-Mate_502443-0870_1x08-1MP_P2.00mm_Vertical
- removed Q2, Q3, Q4, Q5, Q6, Q7, Q8, Q9: AO4407A, AO4407A:SOIC127P600X175-8N
- removed R11, R13, R15, R17, R19, R21, R23: RCT02100KFLF, Resistor_SMD:R_0402_1005Metric
- removed R12, R14, R16, R18, R20, R22, R24: RCT0210KFLF, Resistor_SMD:R_0402_1005Metric
- added C657: CSH0605-101M1CT, Capacitor_SMD:C_Elec_6.3x5.4, F.Cu at (104.3, 147.3)
- added C658: CSH0605-101M1CT, Capacitor_SMD:C_Elec_6.3x5.4, F.Cu at (104.3, 155.5)
- added C659: CSH0605-101M1CT, Capacitor_SMD:C_Elec_6.3x5.4, F.Cu at (104.3, 163.6)
- added D1: XL-1010RGBC-WS2812B, LED_SMD:LED_WS2812B-1010_PLCC4_1.0x1.0mm, F.Cu at (6.38, 14.4)
- added D2: XL-1010RGBC-WS2812B, LED_SMD:LED_WS2812B-1010_PLCC4_1.0x1.0mm, F.Cu at (6.38, 16.8)
- added D3: XL-1010RGBC-WS2812B, LED_SMD:LED_WS2812B-1010_PLCC4_1.0x1.0mm, F.Cu at (6.38, 19.1)
- added D4: XL-1010RGBC-WS2812B, LED_SMD:LED_WS2812B-1010_PLCC4_1.0x1.0mm, F.Cu at (6.38, 21.5)
- C650, C651, C652, C653, C654, C655, C656: value CL21A106KAYNNNE -> CSH0605-101M1CT; footprint Capacitor_SMD:C_0805_2012Metric -> Capacitor_SMD:C_Elec_6.3x5.4
- J1: moved to F.Cu
- moved D1153 298.6 mm to (63.5, 14.4)
- moved D1154 298.6 mm to (63.5, 16.8)
- moved D1201 298.6 mm to (65.9, 14.4)
- moved D1202 298.6 mm to (65.9, 16.8)
- moved D1249 298.6 mm to (68.3, 14.4)
- moved D1250 298.6 mm to (68.3, 16.8)
- moved D1297 298.6 mm to (70.6, 14.4)
- moved D1298 298.6 mm to (70.6, 16.8)
- moved D1729 298.6 mm to (92.1, 14.4)
- moved D1730 298.6 mm to (92.1, 16.8)
- moved D1777 298.6 mm to (94.4, 14.4)
- moved D1778 298.6 mm to (94.4, 16.8)
- moved D1825 298.6 mm to (96.8, 14.4)
- moved D1826 298.6 mm to (96.8, 16.8)
- moved D1873 298.6 mm to (99.2, 14.4)
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Connections:
- C1 pad 1: VDD_S1 -> VDD
- C10 pad 1: VDD_S1 -> VDD
- C11 pad 1: VDD_S1 -> VDD
- C12 pad 1: VDD_S1 -> VDD
- C13 pad 1: VDD_S1 -> VDD
- C14 pad 1: VDD_S1 -> VDD
- C15 pad 1: VDD_S1 -> VDD
- C16 pad 1: VDD_S1 -> VDD
- C17 pad 1: VDD_S1 -> VDD
- C18 pad 1: VDD_S1 -> VDD
- C19 pad 1: VDD_S1 -> VDD
- C2 pad 1: VDD_S1 -> VDD
- C20 pad 1: VDD_S1 -> VDD
- C21 pad 1: VDD_S1 -> VDD
- C22 pad 1: VDD_S1 -> VDD
- C23 pad 1: VDD_S1 -> VDD
- C24 pad 1: VDD_S1 -> VDD
- C25 pad 1: VDD_S1 -> VDD
- C26 pad 1: VDD_S -> VDD
- C27 pad 1: VDD_S -> VDD
- C29 pad 1: VDD_S -> VDD
- C3 pad 1: VDD_S1 -> VDD
- C30 pad 1: VDD_S -> VDD
- C31 pad 1: VDD_S -> VDD
- C32 pad 1: VDD_S -> VDD
- C33 pad 1: VDD_S -> VDD
- C34 pad 1: VDD_S -> VDD
- C35 pad 1: VDD_S1 -> VDD
- C36 pad 1: VDD_S1 -> VDD
- C37 pad 1: VDD_S1 -> VDD
- C38 pad 1: VDD_S1 -> VDD
- C39 pad 1: VDD_S1 -> VDD
- C4 pad 1: VDD_S1 -> VDD
- C40 pad 1: VDD_S1 -> VDD
- C41 pad 1: VDD_S1 -> VDD
- C42 pad 1: VDD_S1 -> VDD
- C43 pad 1: VDD_S1 -> VDD
- C44 pad 1: VDD_S1 -> VDD
- C45 pad 1: VDD_S1 -> VDD
- C46 pad 1: VDD_S1 -> VDD
- C47 pad 1: VDD_S1 -> VDD
- C48 pad 1: VDD_S1 -> VDD
- C49 pad 1: VDD_S1 -> VDD
- C5 pad 1: VDD_S1 -> VDD
- C50 pad 1: VDD_S1 -> VDD
- C51 pad 1: VDD_S1 -> VDD
- C52 pad 1: VDD_S1 -> VDD
- C53 pad 1: VDD_S1 -> VDD
- C54 pad 1: VDD_S1 -> VDD
- C55 pad 1: VDD_S1 -> VDD
- C56 pad 1: VDD_S1 -> VDD
- C57 pad 1: VDD_S1 -> VDD
- C58 pad 1: VDD_S1 -> VDD
- C59 pad 1: VDD_S1 -> VDD
- C6 pad 1: VDD_S1 -> VDD
- C60 pad 1: VDD_S1 -> VDD
- C61 pad 1: VDD_S1 -> VDD
- C62 pad 1: VDD_S1 -> VDD
- C63 pad 1: VDD_S1 -> VDD
- C64 pad 1: VDD_S1 -> VDD
- C65 pad 1: VDD_S1 -> VDD
- C66 pad 1: VDD_S1 -> VDD
- C67 pad 1: VDD_S1 -> VDD
- C68 pad 1: VDD_S1 -> VDD
- C69 pad 1: VDD_S1 -> VDD
- C7 pad 1: VDD_S1 -> VDD
- C70 pad 1: VDD_S1 -> VDD
- C71 pad 1: VDD_S1 -> VDD
- C72 pad 1: VDD_S1 -> VDD
- C73 pad 1: VDD_S1 -> VDD
- C74 pad 1: VDD_S1 -> VDD
- C75 pad 1: VDD_S1 -> VDD
- C76 pad 1: VDD_S1 -> VDD
- C77 pad 1: VDD_S1 -> VDD
- C78 pad 1: VDD_S1 -> VDD
- C79 pad 1: VDD_S1 -> VDD
- C8 pad 1: VDD_S1 -> VDD
- C80 pad 1: VDD_S1 -> VDD
- C81 pad 1: VDD_S1 -> VDD
- C82 pad 1: VDD_S1 -> VDD
- C83 pad 1: VDD_S1 -> VDD
- C84 pad 1: VDD_S1 -> VDD
- C85 pad 1: VDD_S1 -> VDD
- C86 pad 1: VDD_S1 -> VDD
- C87 pad 1: VDD_S1 -> VDD
- C88 pad 1: VDD_S1 -> VDD
- C89 pad 1: VDD_S1 -> VDD
- C9 pad 1: VDD_S1 -> VDD
- D10 pad 2: VDD_S1 -> VDD
- D100 pad 2: VDD_S1 -> VDD
- D101 pad 2: VDD_S1 -> VDD
- D102 pad 2: VDD_S1 -> VDD
- D103 pad 2: VDD_S1 -> VDD
- D104 pad 2: VDD_S1 -> VDD
- D105 pad 2: VDD_S1 -> VDD
- D106 pad 2: VDD_S1 -> VDD
- D107 pad 2: VDD_S1 -> VDD
- D108 pad 2: VDD_S1 -> VDD
- D109 pad 2: VDD_S1 -> VDD
- D11 pad 2: VDD_S1 -> VDD
- D110 pad 2: VDD_S1 -> VDD
- D111 pad 2: VDD_S1 -> VDD
- D112 pad 2: VDD_S1 -> VDD
- D113 pad 2: VDD_S1 -> VDD
- D114 pad 2: VDD_S1 -> VDD
- D115 pad 2: VDD_S1 -> VDD
- D116 pad 2: VDD_S1 -> VDD
- D117 pad 2: VDD_S1 -> VDD
- D118 pad 2: VDD_S1 -> VDD
- D119 pad 2: VDD_S1 -> VDD
- D12 pad 2: VDD_S1 -> VDD
- D120 pad 2: VDD_S1 -> VDD
- D121 pad 2: VDD_S1 -> VDD
- D122 pad 2: VDD_S1 -> VDD
- D123 pad 2: VDD_S1 -> VDD
- D124 pad 2: VDD_S1 -> VDD
- D125 pad 2: VDD_S1 -> VDD
- D126 pad 2: VDD_S1 -> VDD
- D127 pad 2: VDD_S1 -> VDD
- D128 pad 2: VDD_S1 -> VDD
- D129 pad 2: VDD_S1 -> VDD
- D13 pad 2: VDD_S1 -> VDD
- D130 pad 2: VDD_S1 -> VDD
- D131 pad 2: VDD_S1 -> VDD
- D132 pad 2: VDD_S1 -> VDD
- D133 pad 2: VDD_S1 -> VDD
- D134 pad 2: VDD_S1 -> VDD
- D135 pad 2: VDD_S1 -> VDD
- D136 pad 2: VDD_S1 -> VDD
- D137 pad 2: VDD_S1 -> VDD
- D138 pad 2: VDD_S1 -> VDD
- D139 pad 2: VDD_S1 -> VDD
- D14 pad 2: VDD_S1 -> VDD
- D140 pad 2: VDD_S1 -> VDD
- D141 pad 2: VDD_S1 -> VDD
- D142 pad 2: VDD_S1 -> VDD
- D143 pad 2: VDD_S1 -> VDD
- D144 pad 2: VDD_S1 -> VDD
- D145 pad 2: VDD_S1 -> VDD
- D146 pad 2: VDD_S1 -> VDD
- D147 pad 2: VDD_S1 -> VDD
- D148 pad 2: VDD_S1 -> VDD
- D149 pad 2: VDD_S1 -> VDD
- D15 pad 2: VDD_S1 -> VDD
- D150 pad 2: VDD_S1 -> VDD
- D151 pad 2: VDD_S1 -> VDD
- D152 pad 2: VDD_S1 -> VDD
- D153 pad 2: VDD_S1 -> VDD
- D154 pad 2: VDD_S1 -> VDD
- D155 pad 2: VDD_S1 -> VDD
- D156 pad 2: VDD_S1 -> VDD
- D157 pad 2: VDD_S1 -> VDD
- D158 pad 2: VDD_S1 -> VDD
- D159 pad 2: VDD_S1 -> VDD
- D16 pad 2: VDD_S1 -> VDD
- D160 pad 2: VDD_S1 -> VDD
- D161 pad 2: VDD_S1 -> VDD
- D162 pad 2: VDD_S1 -> VDD
- D163 pad 2: VDD_S1 -> VDD
- D164 pad 2: VDD_S1 -> VDD
- D165 pad 2: VDD_S1 -> VDD
- D166 pad 2: VDD_S1 -> VDD
- D167 pad 2: VDD_S1 -> VDD
- D168 pad 2: VDD_S1 -> VDD
- D169 pad 2: VDD_S1 -> VDD
- D17 pad 2: VDD_S1 -> VDD
- D170 pad 2: VDD_S1 -> VDD
- D171 pad 2: VDD_S1 -> VDD
- D172 pad 2: VDD_S1 -> VDD
- D173 pad 2: VDD_S1 -> VDD
- D174 pad 2: VDD_S1 -> VDD
- D175 pad 2: VDD_S1 -> VDD
- D176 pad 2: VDD_S1 -> VDD
- D177 pad 2: VDD_S1 -> VDD
- D178 pad 2: VDD_S1 -> VDD
- D179 pad 2: VDD_S1 -> VDD
- D18 pad 2: VDD_S1 -> VDD
- D180 pad 2: VDD_S1 -> VDD
- D181 pad 2: VDD_S1 -> VDD
- D182 pad 2: VDD_S1 -> VDD
- D183 pad 2: VDD_S1 -> VDD
- D184 pad 2: VDD_S1 -> VDD
- D185 pad 2: VDD_S1 -> VDD
- D186 pad 2: VDD_S1 -> VDD
- D187 pad 2: VDD_S1 -> VDD
- D188 pad 2: VDD_S1 -> VDD
- D189 pad 2: VDD_S1 -> VDD
- D19 pad 2: VDD_S1 -> VDD
- D190 pad 2: VDD_S1 -> VDD
- D191 pad 2: VDD_S1 -> VDD
- D192 pad 2: VDD_S1 -> VDD
- D193 pad 2: VDD_S1 -> VDD
- D194 pad 2: VDD_S1 -> VDD
- D195 pad 2: VDD_S1 -> VDD
- D196 pad 2: VDD_S1 -> VDD
- D197 pad 2: VDD_S1 -> VDD
- D198 pad 2: VDD_S1 -> VDD
- D199 pad 2: VDD_S1 -> VDD
- D20 pad 2: VDD_S1 -> VDD
- D200 pad 2: VDD_S1 -> VDD
- D201 pad 2: VDD_S1 -> VDD
- D202 pad 2: VDD_S1 -> VDD
- D203 pad 2: VDD_S1 -> VDD
- D204 pad 2: VDD_S1 -> VDD
- D205 pad 2: VDD_S1 -> VDD
- D206 pad 2: VDD_S1 -> VDD
- D207 pad 2: VDD_S1 -> VDD
- D208 pad 2: VDD_S1 -> VDD
- D209 pad 2: VDD_S1 -> VDD
- D21 pad 2: VDD_S1 -> VDD
- D210 pad 2: VDD_S1 -> VDD
- D211 pad 2: VDD_S1 -> VDD
- D212 pad 2: VDD_S1 -> VDD
- D213 pad 2: VDD_S1 -> VDD
- D214 pad 2: VDD_S1 -> VDD
- D215 pad 2: VDD_S1 -> VDD
- D216 pad 2: VDD_S1 -> VDD
- D217 pad 2: VDD_S1 -> VDD
- D218 pad 2: VDD_S1 -> VDD
- D219 pad 2: VDD_S1 -> VDD
- D22 pad 2: VDD_S1 -> VDD
- D220 pad 2: VDD_S1 -> VDD
- D221 pad 2: VDD_S1 -> VDD
- D222 pad 2: VDD_S1 -> VDD
- D223 pad 2: VDD_S1 -> VDD
- D224 pad 2: VDD_S1 -> VDD
- D225 pad 2: VDD_S1 -> VDD
- D226 pad 2: VDD_S1 -> VDD
- D227 pad 2: VDD_S1 -> VDD
- D228 pad 2: VDD_S1 -> VDD
- D229 pad 2: VDD_S1 -> VDD
- D23 pad 2: VDD_S1 -> VDD
- D230 pad 2: VDD_S1 -> VDD
- D231 pad 2: VDD_S1 -> VDD
- D232 pad 2: VDD_S1 -> VDD
- D233 pad 2: VDD_S1 -> VDD
- D234 pad 2: VDD_S1 -> VDD
- D235 pad 2: VDD_S1 -> VDD
- D236 pad 2: VDD_S1 -> VDD
- D237 pad 2: VDD_S1 -> VDD
- D238 pad 2: VDD_S1 -> VDD
- D239 pad 2: VDD_S1 -> VDD
- D24 pad 2: VDD_S1 -> VDD
- D240 pad 2: VDD_S1 -> VDD
- D241 pad 2: VDD_S1 -> VDD
- D242 pad 2: VDD_S1 -> VDD
- D243 pad 2: VDD_S1 -> VDD
- D244 pad 2: VDD_S1 -> VDD
- D245 pad 2: VDD_S1 -> VDD
- D246 pad 2: VDD_S1 -> VDD
- D247 pad 2: VDD_S1 -> VDD
- D248 pad 2: VDD_S1 -> VDD
- D249 pad 2: VDD_S1 -> VDD
- D25 pad 2: VDD_S1 -> VDD
- D250 pad 2: VDD_S1 -> VDD
- D251 pad 2: VDD_S1 -> VDD
- D252 pad 2: VDD_S1 -> VDD
- D253 pad 2: VDD_S1 -> VDD
- D254 pad 2: VDD_S1 -> VDD
- D255 pad 2: VDD_S1 -> VDD
- D256 pad 2: VDD_S1 -> VDD
- D257 pad 2: VDD_S1 -> VDD
- D258 pad 2: VDD_S1 -> VDD
- D259 pad 2: VDD_S1 -> VDD
- D26 pad 2: VDD_S1 -> VDD
- D260 pad 2: VDD_S1 -> VDD
- D261 pad 2: VDD_S1 -> VDD
- D262 pad 2: VDD_S1 -> VDD
- D263 pad 2: VDD_S1 -> VDD
- D264 pad 2: VDD_S1 -> VDD
- D265 pad 2: VDD_S1 -> VDD
- D266 pad 2: VDD_S1 -> VDD
- D267 pad 2: VDD_S1 -> VDD
- D268 pad 2: VDD_S1 -> VDD
- D269 pad 2: VDD_S1 -> VDD
- D27 pad 2: VDD_S1 -> VDD
- D270 pad 2: VDD_S1 -> VDD
- D271 pad 2: VDD_S1 -> VDD
- D272 pad 2: VDD_S1 -> VDD
- D273 pad 2: VDD_S1 -> VDD
- D274 pad 2: VDD_S1 -> VDD
- D275 pad 2: VDD_S1 -> VDD
- D276 pad 2: VDD_S1 -> VDD
- D277 pad 2: VDD_S1 -> VDD
- D278 pad 2: VDD_S1 -> VDD
- D279 pad 2: VDD_S1 -> VDD
- D28 pad 2: VDD_S1 -> VDD
- D280 pad 2: VDD_S1 -> VDD
- D281 pad 2: VDD_S1 -> VDD
- D282 pad 2: VDD_S1 -> VDD
- D283 pad 2: VDD_S1 -> VDD
- D284 pad 2: VDD_S1 -> VDD
- D285 pad 2: VDD_S1 -> VDD
- D286 pad 2: VDD_S1 -> VDD
- D287 pad 2: VDD_S1 -> VDD
- D288 pad 2: VDD_S1 -> VDD
- D289 pad 2: VDD_S1 -> VDD
- D29 pad 2: VDD_S1 -> VDD
- D290 pad 2: VDD_S1 -> VDD
- D291 pad 2: VDD_S1 -> VDD
- D292 pad 2: VDD_S1 -> VDD
- D293 pad 2: VDD_S1 -> VDD
- D294 pad 2: VDD_S1 -> VDD
- D295 pad 2: VDD_S1 -> VDD
- D296 pad 2: VDD_S1 -> VDD
- D297 pad 2: VDD_S1 -> VDD
- D298 pad 2: VDD_S1 -> VDD
- D299 pad 2: VDD_S1 -> VDD
- D30 pad 2: VDD_S1 -> VDD
- D300 pad 2: VDD_S1 -> VDD
- D301 pad 2: VDD_S1 -> VDD
- D302 pad 2: VDD_S1 -> VDD
- D303 pad 2: VDD_S1 -> VDD
- D304 pad 2: VDD_S1 -> VDD
- D305 pad 2: VDD_S1 -> VDD
- D306 pad 2: VDD_S1 -> VDD
- D307 pad 2: VDD_S1 -> VDD
- D308 pad 2: VDD_S1 -> VDD
- D309 pad 2: VDD_S1 -> VDD
- D31 pad 2: VDD_S1 -> VDD
- D310 pad 2: VDD_S1 -> VDD
- D311 pad 2: VDD_S1 -> VDD
- D312 pad 2: VDD_S1 -> VDD
- D313 pad 2: VDD_S1 -> VDD
- D314 pad 2: VDD_S1 -> VDD
- D315 pad 2: VDD_S1 -> VDD
- D316 pad 2: VDD_S1 -> VDD
- D317 pad 2: VDD_S1 -> VDD
- D318 pad 2: VDD_S1 -> VDD
- D319 pad 2: VDD_S1 -> VDD
- D32 pad 2: VDD_S1 -> VDD
- D320 pad 2: VDD_S1 -> VDD
- D33 pad 2: VDD_S1 -> VDD
- D34 pad 2: VDD_S1 -> VDD
- D35 pad 2: VDD_S1 -> VDD
- D36 pad 2: VDD_S1 -> VDD
- D37 pad 2: VDD_S1 -> VDD
- D38 pad 2: VDD_S1 -> VDD
- D39 pad 2: VDD_S1 -> VDD
- D40 pad 2: VDD_S1 -> VDD
- D41 pad 2: VDD_S1 -> VDD
- D42 pad 2: VDD_S1 -> VDD
- D43 pad 2: VDD_S1 -> VDD
- D44 pad 2: VDD_S1 -> VDD
- D45 pad 2: VDD_S1 -> VDD
- D46 pad 2: VDD_S1 -> VDD
- D47 pad 2: VDD_S1 -> VDD
- D48 pad 2: VDD_S1 -> VDD
- D49 pad 2: VDD_S1 -> VDD
- D5 pad 2: VDD_S1 -> VDD
- D50 pad 2: VDD_S1 -> VDD
- D51 pad 2: VDD_S1 -> VDD
- D52 pad 2: VDD_S1 -> VDD
- D53 pad 2: VDD_S1 -> VDD
- D54 pad 2: VDD_S1 -> VDD
- D55 pad 2: VDD_S1 -> VDD
- D56 pad 2: VDD_S1 -> VDD
- D57 pad 2: VDD_S1 -> VDD
- D58 pad 2: VDD_S1 -> VDD
- D59 pad 2: VDD_S1 -> VDD
- D6 pad 2: VDD_S1 -> VDD
- D60 pad 2: VDD_S1 -> VDD
- D61 pad 2: VDD_S1 -> VDD
- D62 pad 2: VDD_S1 -> VDD
- D63 pad 2: VDD_S1 -> VDD
- D64 pad 2: VDD_S1 -> VDD
- D65 pad 2: VDD_S1 -> VDD
- D66 pad 2: VDD_S1 -> VDD
- D67 pad 2: VDD_S1 -> VDD
- D68 pad 2: VDD_S1 -> VDD
- D69 pad 2: VDD_S1 -> VDD
- D7 pad 2: VDD_S1 -> VDD
- D70 pad 2: VDD_S1 -> VDD
- D71 pad 2: VDD_S1 -> VDD
- D72 pad 2: VDD_S1 -> VDD
- D73 pad 2: VDD_S1 -> VDD
- D74 pad 2: VDD_S1 -> VDD
- D75 pad 2: VDD_S1 -> VDD
- D76 pad 2: VDD_S1 -> VDD
- D77 pad 2: VDD_S1 -> VDD
- D78 pad 2: VDD_S1 -> VDD
- D79 pad 2: VDD_S1 -> VDD
- D8 pad 2: VDD_S1 -> VDD
- D80 pad 2: VDD_S1 -> VDD
- D81 pad 2: VDD_S1 -> VDD
- D82 pad 2: VDD_S1 -> VDD
- D83 pad 2: VDD_S1 -> VDD
- D84 pad 2: VDD_S1 -> VDD
- D85 pad 2: VDD_S1 -> VDD
- D86 pad 2: VDD_S1 -> VDD
- D87 pad 2: VDD_S1 -> VDD
- D88 pad 2: VDD_S1 -> VDD
- D89 pad 2: VDD_S1 -> VDD
- D9 pad 2: VDD_S1 -> VDD
- D90 pad 2: VDD_S1 -> VDD
- D91 pad 2: VDD_S1 -> VDD
- D92 pad 2: VDD_S1 -> VDD
- D93 pad 2: VDD_S1 -> VDD
- D94 pad 2: VDD_S1 -> VDD
- D95 pad 2: VDD_S1 -> VDD
- D96 pad 2: VDD_S1 -> VDD
- D97 pad 2: VDD_S1 -> VDD
- D98 pad 2: VDD_S1 -> VDD
- D99 pad 2: VDD_S1 -> VDD
- U2 pad 5: VDD_S -> VDD
- U3 pad 5: VDD_S -> VDD
- U4 pad 5: VDD_S -> VDD
- U5 pad 5: VDD_S -> VDD
- U6 pad 5: VDD_S -> VDD
- U7 pad 5: VDD_S -> VDD
- U8 pad 5: VDD_S -> VDD
- U9 pad 5: VDD_S -> VDD
