File: cad/led_bage.kicad_pcb (KiCad board)
At the start: 4 copper layers, 72.6 x 123.7 mm, 3238 parts, among them J1 Conn_01x08_Socket, U2 74AHCT1G125, U3 74AHCT1G125, U4 74AHCT1G125, U5 74AHCT1G125, U6 74AHCT1G125, U7 74AHCT1G125, U8 74AHCT1G125, U9 74AHCT1G125

Commit message: feat: lay down 40x64 LED grid with fanout and decoupling
Place 2560 LEDs in a 40-col x 64-row serpentine grid (8 data chains of
320 LEDs each, snake continues across chain boundaries -- matches the
sample's D50/D51 transition pattern).

Drop C642..C649 from the schematic to bring the 0603 cap count from 648
down to 640, matching the 20x32 = 640 2x2 LED-block count of the new
grid (the previous 54x48 layout had 648 blocks).

Run the LED-grid pipeline against the main board:
- normalize LED rotation to 0 deg (idempotent)
- 5120 power fanout vias placed on VDD_S / GND
- 640 decoupling caps snapped to block centers on B.Cu, rotated 45 deg

New: place_leds.py -- parameterized serpentine grid layout, defaults to
keeping D1 at its existing position so the grid can be repositioned by
moving D1 alone.

Bug fixes to existing pipeline scripts:
- add_power_vias.py: filter by net name (VDD/VDD_S/GND) instead of pad
  pin function, since the LED footprint uses VDD_2 / GND_3 pin names.
- snap_caps_to_blocks.py: when in-area cap count != block count but the
  total 0603 cap count matches, fall back to using all 0603 caps. Handles
  the typical post-sync state where caps are still piled in the import
  cluster.
Parts:
- removed C642, C643, C644, C645, C646, C647, C648, C649: CL21B105KAFNNNE, Capacitor_SMD:C_0603_1608Metric
- C1, C10, C100, C101, C102, C103, C104, C105, C106, C107, C108, C109, C11, C110, C111, C112, C113, C114, C115, C116, C117, C118, C119, C12, C120, C121, C122, C123, C124, C125, C126, C127, C128, C129, C13, C130, C131, C132, C133, C134, C135, C136, C137, C138, C139, C14, C140, C141, C142, C143, C144, C145, C146, C147, C148, C149, C15, C150, C151, C152, C153, C154, C155, C156, C157, C158, C159, C16, C160, C161, C162, C163, C164, C165, C166, C167, C168, C169, C17, C170, C171, C172, C173, C174, C175, C176, C177, C178, C179, C18, C180, C181, C182, C183, C184, C185, C186, C187, C188, C189, C19, C190, C191, C192, C193, C194, C195, C196, C197, C198, C199, C2, C20, C200, C201, C202, C203, C204, C205, C206, C207, C208, C209, C21, C210, C211, C212, C213, C214, C215, C216, C217, C218, C219, C22, C220, C221, C222, C223, C224, C225, C226, C227, C228, C229, C23, C230, C231, C232, C233, C234, C235, C236, C237, C238, C239, C24, C240, C241, C242, C243, C244, C245, C246, C247, C248, C249, C25, C250, C251, C252, C253, C254, C255, C256, C257, C258, C259, C26, C260, C261, C262, C263, C264, C265, C266, C267, C268, C269, C27, C270, C271, C272, C273, C274, C275, C276, C277, C278, C279, C280, C281, C282, C283, C284, C285, C286, C287, C288, C289, C29, C290, C291, C292, C293, C294, C295, C296, C297, C298, C299, C3, C30, C300, C301, C302, C303, C304, C305, C306, C307, C308, C309, C31, C310, C311, C312, C313, C314, C315, C316, C317, C318, C319, C32, C320, C321, C322, C323, C324, C325, C326, C327, C328, C329, C33, C330, C331, C332, C333, C334, C335, C336, C337, C338, C339, C34, C340, C341, C342, C343, C344, C345, C346, C347, C348, C349, C35, C350, C351, C352, C353, C354, C355, C356, C357, C358, C359, C36, C360, C361, C362, C363, C364, C365, C366, C367, C368, C369, C37, C370, C371, C372, C373, C374, C375, C376, C377, C378, C379, C38, C380, C381, C382, C383, C384, C385, C386, C387, C388, C389, C39, C390, C391, C392, C393, C394, C395, C396, C397, C398, C399, C4, C40, C400, C401, C402, C403, C404, C405, C406, C407, C408, C409, C41, C410, C411, C412, C413, C414, C415, C416, C417, C418, C419, C42, C420, C421, C422, C423, C424, C425, C426, C427, C428, C429, C43, C430, C431, C432, C433, C434, C435, C436, C437, C438, C439, C44, C440, C441, C442, C443, C444, C445, C446, C447, C448, C449, C45, C450, C451, C452, C453, C454, C455, C456, C457, C458, C459, C46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: moved to B.Cu
- moved D2401 153.8 mm to (6.38, 111.9)
- moved D2402 151.1 mm to (7.95, 111.9)
- moved D2403 148.4 mm to (9.51, 111.9)
- moved D2404 145.7 mm to (11.1, 111.9)
- moved D2545 145.0 mm to (29.8, 116.8)
- moved D2546 144.5 mm to (28.3, 116.8)
- moved D2547 144.0 mm to (26.7, 116.8)
- moved D2548 143.6 mm to (25.1, 116.8)
- moved D2549 143.2 mm to (23.6, 116.8)
- moved D2405 143.0 mm to (12.6, 111.9)
- moved D2550 142.9 mm to (22.0, 116.8)
- moved D2560 142.7 mm to (6.38, 116.8)
- moved D2551 142.6 mm to (20.4, 116.8)
- moved D2559 142.5 mm to (7.95, 116.8)
- moved D2552 142.4 mm to (18.9, 116.8)
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Routing:
- net VDD: vias 0 -> 2560
- net GND: vias 0 -> 2560
