File: cad/led_bage.kicad_pcb (KiCad board)
At the start: 6 copper layers, 91.1 x 134.1 mm, 3235 parts, among them J1 Conn_01x08_Socket, J2 Conn_01x10_MountingPin, U1 SI7145DP-T1-GE3, U2 74AHCT1G125, U3 74AHCT1G125, U4 74AHCT1G125, U5 74AHCT1G125, U6 74AHCT1G125, U7 74AHCT1G125, U8 74AHCT1G125, U9 74AHCT1G125

Commit message: feat(cad): rounded 71x150 mm outline with lanyard holes and J2 top band
- Edge.Cuts: plain rounded rectangle, R5 corners, no tabs.
- H1/H2: 5 mm plated lanyard holes with GND ring, board-only footprints.
- J2 centered in a new 16 mm top band, cable still exits the top edge.
- Power entry re-laid with F/B VDD pours and a 24-via VDD_S field,
  following the U1 drain/source fix.
- redesign_top_band.py generates it idempotently; test_board.py checks
  outline, holes, U1 nets, PTH mask openings and DRC with schematic parity.
Parts:
- H1, H2: value MountingHole_3.5mm -> Lanyard_Eyelet_5mm; footprint MountingHole_3.5mm -> (none)
- moved J2 22.1 mm to (19.0, -4.30)
- moved H1 19.3 mm to (7.80, -13.2)
- moved H2 19.3 mm to (65.9, -13.2)
Connections:
- R3 pad 1: VDD -> VDD_S
- U1 pad 1: VDD -> VDD_S
- U1 pad 2: VDD -> VDD_S
- U1 pad 3: VDD -> VDD_S
- U1 pad 5: VDD_S -> VDD
- U1 pad 6: VDD_S -> VDD
- U1 pad 7: VDD_S -> VDD
- U1 pad 8: VDD_S -> VDD
Routing:
- net VDD: track 81.0 -> 0.00 mm, vias 0 -> 13
- net VDD_S: track 2010.3 -> 2011.8 mm, vias 2611 -> 2622
- net GND: vias 2606 -> 2609
- added copper zone on B.Cu, net VDD
- added copper zone on F.Cu, net VDD
- added copper zone on F.Cu, net VDD_S
Other:
- board size 91.1 x 134.1 mm -> 71.1 x 150.1 mm
