File: cad/led_bage.kicad_sch (KiCad schematic)
At the start: 3233 parts, among them J1 Conn_01x08_Socket, J2 Conn_01x10_MountingPin, U1 SI7145DP-T1-GE3, U2 74AHCT1G125, U3 74AHCT1G125, U4 74AHCT1G125, U5 74AHCT1G125, U6 74AHCT1G125, U7 74AHCT1G125, U8 74AHCT1G125, U9 74AHCT1G125

Commit message: feat: rename LEDs per chain (DA..DH), add lanyard tabs, 6-layer stackup
Renumber LED refs from sequential D1..D2560 (which broke JLC's <=2048
ref-number cap on chain 8) to per-chain letter prefix DA1..DH320. Both
schematic and PCB updated in lockstep via cad/renumber_leds.py. Also
fixes the stale D2561 -> TVS1 sync that didn't propagate from the
schematic.

Add side tabs at top corners (10x12 mm, 3.5 mm hole each) for lanyard
mounting. Currently T-shaped (top edge merged with main board) and
bare-FR4 hole — flagged for structural redesign next session.

Move to 6-layer stackup: F | GND | VDD_S | VDD_S | GND | B. Existing
through-vias automatically pick up the duplicate inner planes; halves
both VDD_S and GND DC impedances. All 4 inner zones at 0.15 mm
clearance / 0.15 mm min thickness, single continuous fill region each.
Parts:
- renumbered D1 to DA1, D10 to DA10, D100 to DA100, D101 to DA101, D102 to DA102, D103 to DA103, D104 to DA104, D105 to DA105, D106 to DA106, D107 to DA107, D108 to DA108, D109 to DA109, D11 to DA11, D110 to DA110, D111 to DA111, D112 to DA112, D113 to DA113, D114 to DA114, D115 to DA115, D116 to DA116, D117 to DA117, D118 to DA118, D119 to DA119, D12 to DA12, D120 to DA120, D121 to DA121, D122 to DA122, D123 to DA123, D124 to DA124, D125 to DA125, D126 to DA126, D127 to DA127, D128 to DA128, D129 to DA129, D13 to DA13, D130 to DA130, D131 to DA131, D132 to DA132, D133 to DA133, D134 to DA134, D135 to DA135, D136 to DA136, D137 to DA137, D138 to DA138, D139 to DA139, D14 to DA14, D140 to DA140, D141 to DA141, D142 to DA142, D143 to DA143, D144 to DA144, D145 to DA145, D146 to DA146, D147 to DA147, D148 to DA148, D149 to DA149, D15 to DA15, D150 to DA150, D151 to DA151, D152 to DA152, D153 to DA153, D154 to DA154, D155 to DA155, D156 to DA156, D157 to DA157, D158 to DA158, D159 to DA159, D16 to DA16, D160 to DA160, D161 to DA161, D162 to DA162, D163 to DA163, D164 to DA164, D165 to DA165, D166 to DA166, D167 to DA167, D168 to DA168, D169 to DA169, D17 to DA17, D170 to DA170, D171 to DA171, D172 to DA172, D173 to DA173, D174 to DA174, D175 to DA175, D176 to DA176, D177 to DA177, D178 to DA178, D179 to DA179, D18 to DA18, D180 to DA180, D181 to DA181, D182 to DA182, D183 to DA183, D184 to DA184, D185 to DA185, D186 to DA186, D187 to DA187, D188 to DA188, D189 to DA189, D19 to DA19, D190 to DA190, D191 to DA191, D192 to DA192, D193 to DA193, D194 to DA194, D195 to DA195, D196 to DA196, D197 to DA197, D198 to DA198, D199 to DA199, D2 to DA2, D20 to DA20, D200 to DA200, D201 to DA201, D202 to DA202, D203 to DA203, D204 to DA204, D205 to DA205, D206 to DA206, D207 to DA207, D208 to DA208, D209 to DA209, D21 to DA21, D210 to DA210, D211 to DA211, D212 to DA212, D213 to DA213, D214 to DA214, D215 to DA215, D216 to DA216, D217 to DA217, D218 to DA218, D219 to DA219, D22 to DA22, D220 to DA220, D221 to DA221, D222 to DA222, D223 to DA223, D224 to DA224, D225 to DA225, D226 to DA226, D227 to DA227, D228 to DA228, D229 to DA229, D23 to DA23, D230 to DA230, D231 to DA231, D232 to DA232, D233 to DA233, D234 to DA234, D235 to DA235, D236 to DA236, D237 to DA237, D238 to DA238, D239 to DA239, D24 to DA24, D240 to DA240, D241 to DA241, D242 to DA242, D243 to DA243, D244 to DA244, D245 to DA245, D246 to DA246, D247 to DA247, D248 to DA248, D249 to DA249, D25 to DA25, D250 to DA250, D251 to DA251, D252 to DA252, D253 to DA253, D254 to DA254, D255 to DA255, D256 to DA256, D257 to DA257, D258 to DA258, D259 to DA259, D26 to DA26, D260 to DA260, D261 to DA261, D262 to DA262, D263 to DA263, D264 to DA264, D265 to DA265, D266 to DA266, D267 to DA267, D268 to DA268, D269 to DA269, D27 to DA27, D270 to DA270, D271 to DA271, D272 to DA272, D273 to DA273, D274 to DA274, D275 to DA275, D276 to DA276, D277 to DA277, D278 to DA278, D279 to DA279, D28 to DA28, D280 to DA280, D281 to DA281, D282 to DA282, D283 to DA283, D284 to DA284, D285 to DA285, D286 to DA286, D287 to DA287, D288 to DA288, D289 to DA289, D29 to DA29, D290 to DA290, D291 to DA291, D292 to DA292, D293 to DA293, D294 to DA294, D295 to DA295, D296 to DA296, D297 to DA297, D298 to DA298, D299 to DA299, D3 to DA3, D30 to DA30, D300 to DA300, D301 to DA301, D302 to DA302, D303 to DA303, D304 to DA304, D305 to DA305, D306 to DA306, D307 to DA307, D308 to DA308, D309 to DA309, D31 to DA31, D310 to DA310, D311 to DA311, D312 to DA312, D313 to DA313, D314 to DA314, D315 to DA315, D316 to DA316, D317 to DA317, D318 to DA318, D319 to DA319, D32 to DA32, D320 to DA320, D33 to DA33, D34 to DA34, D35 to DA35, D36 to DA36, D37 to DA37, D38 to DA38, D39 to DA39, D4 to DA4, D40 to DA40, D41 to DA41, D42 to DA42, D43 to DA43, D44 to DA44, D45 to DA45, D46 to DA46, D47 to DA47, D48 to DA48, D49 to DA49, D5 to DA5, D50 to DA50, D51 to DA51, D52 to DA52, D53 to DA53, D54 to DA54, D55 to DA55, D56 to DA56, D57 to DA57, D58 to DA58, D59 to DA59, D6 to DA6, D60 to DA60, D61 to DA61, D62 to DA62, D63 to DA63, D64 to DA64, D65 to DA65, D66 to DA66, D67 to DA67, D68 to DA68, D69 to DA69, D7 to DA7, D70 to DA70, D71 to DA71, D72 to DA72, D73 to DA73, D74 to DA74, D75 to DA75, D76 to DA76, D77 to DA77, D78 to DA78, D79 to DA79, D8 to DA8, D80 to DA80, D81 to DA81, D82 to DA82, D83 to DA83, D84 to DA84, D85 to DA85, D86 to DA86, D87 to DA87, D88 to DA88, D89 to DA89, D9 to DA9, D90 to DA90, D91 to DA91, D92 to DA92, D93 to DA93, D94 to DA94, D95 to DA95, D96 to DA96, D97 to DA97, D98 to DA98, D99 to DA99, D321 to DB1, D330 to DB10, D420 to DB100, D421 to DB101, D422 to DB102, D423 to DB103, D424 to DB104, D425 to DB105, D426 to DB106, D427 to DB107, D428 to DB108, D429 to DB109, D331 to DB11, D430 to DB110, D431 to DB111, D432 to DB112, D433 to DB113, D434 to DB114, D435 to DB115, D436 to DB116, D437 to DB117, D438 to DB118, D439 to DB119, D332 to DB12, D440 to DB120, D441 to DB121, D442 to DB122, D443 to DB123, D444 to DB124, D445 to DB125, D446 to DB126, D447 to DB127, D448 to DB128, D449 to DB129, D333 to DB13, D450 to DB130, D451 to DB131, D452 to DB132, D453 to DB133, D454 to DB134, D455 to DB135, D456 to DB136, D457 to DB137, D458 to DB138, D459 to DB139, D334 to DB14, D460 to DB140, D461 to DB141, D462 to DB142, D463 to DB143, D464 to DB144, D465 to DB145, D466 to DB146, D467 to DB147, D468 to DB148, D469 to DB149, D335 to DB15, D470 to DB150, D471 to DB151, D472 to DB152, D473 to DB153, D474 to DB154, D475 to DB155, D476 to DB156, D477 to DB157, D478 to DB158, D479 to DB159, D336 to DB16, D480 to DB160, D481 to DB161, D482 to DB162, D483 to DB163, D484 to DB164, D485 to DB165, D486 to DB166, D487 to DB167, D488 to DB168, D489 to DB169, D337 to DB17, D490 to DB170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
