File: cad/led_bage_sample/led_bage_sample.kicad_sch (KiCad schematic)
At the start: 136 parts, among them J1 Conn_01x06, Q2 AO4407A, U1 74AHCT1G125, U2 74AHCT1G125

Commit message: feat: scale protection circuit toward 2500-LED main board
Add Si7145DP P-FET (U1) and SnapEDA-imported library table (fp-lib-table)
to the main board. WIP: U1 pin-to-net mapping is incorrect — drain pads
currently land on VDD instead of VDD_S, so the FET is shorted across
itself and not actually protecting anything yet.

Add three pcbnew automation scripts to support the build:
- stitch_power_planes.py: checkerboard via stitching across In1.Cu/In2.Cu
- add_thermal_vias.py: drops thermal via grid under exposed pads
- place_bulk_caps.py: clones a template cap across the LED bbox

Sample board updated alongside the main board for prototyping continuity.
Connections:
- net GND: now also C25.2; no longer C25.1
- net VDD_S: now also C25.1; no longer C25.2
